Commit message: Update wsg32 urdf

File: src/pb_robot/models/wsg32_description/wsg_32.urdf (robot description, URDF)
Before this commit: robot wsg_32, 5 links, 4 joints
Links:
- removed link base_link
- removed link finger_left
- removed link finger_right
- removed link gripper_left
- removed link gripper_right
- added link hand_link, mass 0.19187770361295; collision mesh filename=package://wsg32_description/meshes/hand_link.STL; visual mesh filename=package://wsg32_description/meshes/hand_link.STL
- added link left_universal_finger_link, mass 0.001; collision mesh filename=package://wsg32_description/meshes/stub.obj scale=0.001; visual mesh filename=package://wsg32_description/meshes/stub.obj scale=0.001
- added link right_universal_finger_link, mass 0.001; collision mesh filename=package://wsg32_description/meshes/stub.obj scale=0.001; visual mesh filename=package://wsg32_description/meshes/stub.obj scale=0.001
- added link wsg_50_gripper_base_link_gripper_left, mass 3.41920163633724E-06; collision mesh filename=package://wsg32_description/meshes/left_finger_link.STL; visual mesh filename=package://wsg32_description/meshes/left_finger_link.STL
- added link wsg_50_gripper_base_link_gripper_right, mass 3.41920163633724E-06; collision mesh filename=package://wsg32_description/meshes/right_finger_link.STL; visual mesh filename=package://wsg32_description/meshes/right_finger_link.STL
Joints:
- removed joint base_joint_gripper_left
- removed joint base_joint_gripper_right
- removed joint guide_joint_finger_left
- removed joint guide_joint_finger_right
- added joint left_universal_finger_joint: type fixed, parent wsg_50_gripper_base_link_gripper_left, child left_universal_finger_link, origin xyz=0.00755 -0.0045 0 rpy=0 3.14159 -1.57079
- added joint right_universal_finger_joint: type fixed, parent wsg_50_gripper_base_link_gripper_right, child right_universal_finger_link, origin xyz=0.00755 0.0 0.0049 rpy=0 -1.57079 -1.57079
- added joint wsg_50_gripper_base_joint_gripper_left: type prismatic, parent hand_link, child wsg_50_gripper_base_link_gripper_left, origin xyz=-0.0003903 -0.0078 0.069014 rpy=3.1416 -1.5708 0, axis 0 -1 0, limit lower=-0.028 upper=0 effort=0 velocity=0
- added joint wsg_50_gripper_base_joint_gripper_right: type prismatic, parent hand_link, child wsg_50_gripper_base_link_gripper_right, origin xyz=-0.0003903 0.0078 0.069012 rpy=-1.5708 -1.5708 0, axis 0 0 1, limit lower=0 upper=0.028 effort=0 velocity=0
